Commit message: Improve RTF

File: so_arm100_gym_description/models/so_arm100/so100.urdf (robot description, URDF)
Before this commit: robot so_arm100, 10 links, 9 joints
Links:
- link base: geometry collision box size=0.1 0.1 0.1; visual mesh filename=package://so_arm100_gym_description/models/so_arm100/assets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
- link gripper: geometry collision box size=0.05 0.105 0.065; visual mesh filename=package://so_arm100_gym_description/models/so_arm100/assets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
- link jaw: geometry collision box size=0.025 0.09 0.05; visual mesh filename=package://so_arm100_gym_description/models/so_arm100/assets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
- link lower_arm: geometry collision box size=0.06 0.04 0.12; visual mesh filename=package://so_arm100_gym_description/models/so_arm100/assets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
- link shoulder: geometry collision box size=0.06 0.09 0.065; visual mesh filename=package://so_arm100_gym_description/models/so_arm100/assets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
- link upper_arm: geometry collision box size=0.08 0.1535 0.025; visual mesh filename=package://so_arm100_gym_description/models/so_arm100/assets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
- link wrist: geometry collision box size=0.065 0.075 0.035; visual mesh filename=package://so_arm100_gym_description/models/so_arm100/assets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
